File: hw/analog-out/analog-out.sch (EAGLE design)
At the start: 126 parts

Commit message: First verision of dac schematic
Parts:
- removed ADC_: LTC2312, LTC2312-14:LTC2312ITS8-14TRMPBF
- removed ADC_IN, ADC_REF, A_IN, FILTER, REF_2.048: TESTPIN, myLib:TESTPIN
- removed ANALOG_IN: PTR1B1,27, testpad:PTR1B1,27
- removed C15, C18, C19: 2u2, rcl:C-EUC0805K
- removed C8: 100n, rcl:C-EUC0805K
- removed C_FILTER: 330p, rcl:C-EUC0805K
- removed C_FILTER1: nb, rcl:C-EUC0805K
- removed INSTR_AMP: AD8250ARMZ, parts:AD8250ARMZ
- removed LED2: GREEN, led:LEDSML0805
- removed MINUS, PLUS: 23.3200-21, CONN_BANANA_JACK_4MM_STAUBLI:23.3200-21
- removed MOV1: CV300CVQ300K10BL1, myLib:CV300CVQ300K10BL1
- removed PIN_HEADER_SMD: (no value), SMD10_2_pinheader:MA05-2
- removed R11: 0, rcl:R-EU_R0805
- removed R12: 47k, rcl:R-EU_R0805
- removed R13: inf, rcl:R-EU_R0805
- removed R14, R_FILTER1: nb, rcl:R-EU_R0805
- removed R53, R57, R58: nb, rcl:R-EU_R1206
- removed R_FILTER: 2k2, rcl:R-EU_R0805
- added C27: 10p, rcl:C-EUC0805
- added C28, C29: 100n, rcl:C-EUC0805
- added CONV1: PTR1B1,27, testpad:PTR1B1,27
- added POWER1: gr, led:LEDSML0805
- added R23: 680, resistor:R-EU_R0805
- added REF_2.5: TESTPIN, myLib:TESTPIN
- added U$3: ADA4522-2ARZ-RL, my:ADA4522-2ARZ-RL
- added U$4: MAX1036EKA+T, my:MAX1036EKA+T
- added U$5: 73099RED, my:73099RED
- added U$6: 73099BLACK, my:73099BLACK
- C5: device rcl:C-EUC0805K -> rcl:C-EUC0805; MOUSER (none) -> 81-GRM21BZ71E106KE5L
- R10: value 390k -> tbd; DIGIKEY 2019-RK73H2ATTD3903FTR-ND -> Y1629-120DTR-ND
- R3: value 680 -> tbd; DIGIKEY A129747TR-ND -> Y1629-120DTR-ND; MOUSER 652-CR0805JW-561ELF -> (none)
- R4, R5: value nb -> tbd; device rcl:R-EU_R1206 -> rcl:R-EU_R0805; DIGIKEY (none) -> Y1629-120DTR-ND; MOUSER check config -> (none)
- REF: DIGIKEY 161-LT6654BHS6-2.048#WTRPBFTR-ND -> 505-LT6654AIS6-2.5#TRMPBFTR-ND
- U$1: value 0508.500MXEP -> LTC2642IMS-16; device 0508.500MXEP.FUSE:0508.500MXEP -> my:LTC2642IMS-16; DIGIKEY 283-4458-1-ND -> (none)
- U$2: DIGIKEY (none) -> 296-40574-2-ND
Connections:
- removed net >ADC: ADC_A.AIN, ADC_IN.1, C_FILTER.1, R10.2, R11.2, R_FILTER.1
- removed net CONV<: PIN_HEADER_SMD.6, RJ45.5
- removed net CONV>: CONVERSIONA.VIN, PIN_HEADER_SMD.1
- removed net GAIN_LSB: INSTR_AMPA.A0, U$2.P6
- removed net GAIN_MSB: INSTR_AMPA.A1, U$2.P7
- removed net N$18: R11.1, R13.2, SATURATION_DETECTA.INA+
- removed net N$20: ANALOG_IN.TP, A_IN.1, R14.2, R4.1, U$20G$1.NC
- removed net N$21: R57.1, R58.2
- removed net N$29: R4.2, R53.1
- removed net N$4: I2CA.SCL1, R18.1, ROHM_I2CG$1.SCL, U$2.SCL
- removed net N$6: I2CA.SDA1, R19.1, ROHM_I2CG$1.SDA, U$2.SDA
- removed net N$66: R53.2, R58.1
- removed net N$67: R5.1, R57.2
- removed net N$8: ADC_G$1.REF, ADC_REF.1, C19.2
- removed net N_STATUS_LED: R8.1, U$2.P2
- removed net SAT_DETECT: R3.1, SATURATION_DETECTA.OUTA, SATURATION_DETECTA.OUTB, U$2.P5
- removed net SCL<: PIN_HEADER_SMD.5, RJ45.7
- removed net SCL>: I2CA.SCL2, PIN_HEADER_SMD.2, R22.1
- removed net SDO<: PIN_HEADER_SMD.4, RJ45.8
- removed net SDO>: I2CA.SDA2, PIN_HEADER_SMD.3, R20.1
- new net ANALOG_FEEDBACK: U$20G$1.COM, U$4G$1.AIN0
- new net CONV: CONV1.TP, CONVERSIONA.VIN, RJ45.5
- new net N$22: R8.1, STATUS.A
- new net N$27: POWER1.A, R23.1
- new net SCL: I2CA.SCL2, R22.1, RJ45.7
- new net SDO: I2CA.SDA2, R20.1, RJ45.8
- new net STATUS_LED: R8.2, U$2.P2
- new net V_OUT: R10.1, R4.2, TP1.PP, TP3.PP, U$3G$2.OUT, U$5.P$1
- net +5V: now also C28.1, C29.1, C5.1, R23.2, U$1G$2.VCC, U$3G$3.VEE, U$4G$2.VCC; no longer ADC_G$1.OVDD, ADC_G$1.VDD, C15.1, C18.1, C5.2, INSTR_AMPG$1.+VS, LED2.A, STATUS.A
- net -5V: now also C28.2, U$3G$3.VCC; no longer C8.2, INSTR_AMPG$1.-VS
- net CONV_ADC: now also U$1G$1.!CS; no longer ADC_A.CONV
- net DGND: now also C29.2, C5.2, POWER1.C, R3.2, R5.2, STATUS.C, U$1G$2.GND, U$4G$2.VEE, U$6.P$1; no longer ADC_G$1.GND, C15.2, C18.2, C19.1, C5.1, C8.1, C_FILTER.2, C_FILTER1.2, INSTR_AMPA.-IN, INSTR_AMPG$1.DGND, MINUS.1, MOV1.2, R12.1, R13.1, R14.1
- net N$1: now also C27.2, U$1G$1.INV, U$3G$1.-IN; no longer INSTR_AMPA.OUT, R_FILTER.2
- net N$14: now also I2CA.SDA1, R19.1, ROHM_I2CG$1.SDA, U$2.SDA, U$4G$1.SDA; no longer LED2.C, R3.2
- net N$15: now also R4.1, R5.1, U$3G$2.-IN; no longer C_FILTER1.1, INSTR_AMPA.+IN, R_FILTER1.1
- net N$16: now also R10.2, R3.1, U$20G$1.NC; no longer PLUS.1, TP1.PP, TP3.PP, U$1.IN
- net N$17: now also I2CA.SCL1, R18.1, ROHM_I2CG$1.SCL, U$2.SCL, U$4G$1.SCL; no longer R10.1, R12.2, SATURATION_DETECTA.INB-
- net N$26: now also SCK.2, SCK_A.TP, U$1G$1.SCLK; no longer R8.2, STATUS.C
- net N$5: now also U$1G$1.VOUT, U$3G$1.+IN; no longer FILTER.1, R_FILTER1.2, U$20G$1.COM
- net N$9: now also C27.1, U$1G$1.RFB, U$3G$1.OUT, U$3G$2.+IN; no longer MOV1.1, R5.2, U$1.OUT
- net N_WE: no longer INSTR_AMPA.!WR
- net REF_: now also REF_2.5.1, U$1G$1.REF; no longer INSTR_AMPA.REF, REF_2.048.1
- net SCK_ADC: no longer ADC_A.SCK, SCK.2, SCK_A.TP
- net SDO_ADC: now also U$1G$1.DIN; no longer ADC_A.SDO
Other:
- note added: "Address: 0b0100000"
- note added: "Address: 0b101000X"
- note added: "Address: 0b1100100"
- note added: "Amplifiaction needs to be defined"
- note added: "Feedback circuit"
- note added: "Make sure no negative volatages can appear on AIN!!"
- note added: "What is !CRL needed for?"
- note removed: "100mA, 250V"
- note removed: "200kHz = 2.2k + 360p"
- note removed: "220kHz = 2.2k + 330p"
- moved on the sheet: C1, C5, C51, GND1, GND2, GND3, GND5, R10, R3, R4, R5, R8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

Commit message: first revision of dac board
Signed-off-by: Manuel Pitz <manuel.pitz@eonerc.rwth-aachen.de>
Parts:
- removed 74LVC1G11: SN74LVC1G32DCKT, 74LVC1G11DBV:SN74LVC1G11DBVRDBV0006A_L
- removed C16, C17, C21, C26: 100n, rcl:C-EUC0805K
- removed CONV_A, CONV_T, GND1, GND2, GND3, SCK_A, SCK_T, SDO_A, SDO_T: PTR1B1,27, testpad:PTR1B1,27
- removed FLIP-FLOP: 74HC74PW, 74H74PW:74HC74PW-Q100,118
- removed R10: tbd, rcl:R-EU_R0805
- removed SATURATION_DETECT: ADCMP670, ADCMP670:ADCMP670-1YUJZ-RL7
- removed SDO: (no value), con-lstb:MA03-1
- removed SN74LVC1G32: 74LVC1G32, SN74LVC1G32:SN74LVC1G32DCKTDCK5-M
- removed U$20: MAX4564UMAX, myLib:MAX4564UMAX
- added +12V: TESTPIN, myLib:TESTPIN
- added C15, C18, C19: tbd, rcl:C-EUC0805K
- added C8: 1u, rcl:C-EUC0805K
- added CONV_TP, SCK_TP, SDA_TP: PTR1B1,27, testpad:PTR1B1,27
- added R11: 10k, rcl:R-TRIMMT93YA
- added R12: 100, resistor:R-EU_R0805
- added SDA: (no value), jumper:JP1E
- added U$11: MAX4659, my:MAX4659
- added U$7: LDO_MIC5233-5.0YM5-TR, my:LDO_MIC5233-5.0YM5-TR
- added U$8, U$9: 4u7, my:NRS5010T4R7MMGF
- C2: value 100n -> 1u
- C20: value 100n -> tbd
- C22, C25: device rcl:C-EUC0805K -> rcl:C-EUC0805; MOUSER (none) -> 81-GRM21BZ71E106KE5L
- CONV, SCK: device con-lstb:MA03-1 -> jumper:JP1E; DIGIKEY 732-5316-ND -> (none)
- DC-DC_CONVERTER: DIGIKEY TDN3-1221WISM-ND -> TDN3-1222WISM-ND; MANUFACTURER_PART_NUMBER TDN 3-1221WISM -> (none); MOUSER (none) -> 495-TDN3-1222WISM
- R3: value tbd -> 1k
- R4: value tbd -> 10k; device rcl:R-EU_R0805 -> rcl:R-TRIMMT93YA; DIGIKEY Y1629-120DTR-ND -> (none)
- R5: value tbd -> 2k2
- renumbered -5V to -12V
Connections:
- removed net -5V: -12V.1, C17.2, C21.2, C24.2, C28.2, DC-DC_CONVERTER.-VOUT, U$20G$2.V-, U$3G$3.VCC
- removed net ANALOG_FEEDBACK: U$20G$1.COM, U$4G$1.AIN0
- removed net N$23: 74LVC1G11A.B, FLIP-FLOPA.2Q
- removed net N$25: CONV.3, FLIP-FLOPA.1D
- removed net N$30: SDO.2, SDO_T.TP, SERIAL_DATAA.TXD
- removed net N$31: SDO.3, SN74LVC1G32A.Y
- new net +12V: +12V.1, C15.1, C22.2, C28.1, C8.1, U$11G$1.VCC, U$3G$3.VEE, U$7.EN, U$7.IN, U$8.1
- new net -12V: -12V.1, C20.2, C25.1, C28.2, U$11G$1.VSS, U$3G$3.VCC, U$9.1
- new net N$18: R12.2, U$11G$2.COM
- new net N$4: SDA.2, SERIAL_DATAA.TXD
- new net N$6: C19.2, C24.2, DC-DC_CONVERTER.-VOUT, U$9.2
- net +5V: now also U$1G$1.!CLR, U$7.OUT; no longer 74LVC1G11G$1.VCC, C16.1, C20.2, C22.1, C25.1, C26.1, C28.1, DC-DC_CONVERTER.+VOUT, FLIP-FLOPA.1RD, FLIP-FLOPA.1SD, FLIP-FLOPA.2RD, FLIP-FLOPA.2SD, FLIP-FLOPSUPPLY.VCC, SATURATION_DETECTB.VDD1, SN74LVC1G32G$1.VCC, U$20G$2.V+, U$3G$3.VEE
- net CONV_ADC: now also CONV_TP.TP; no longer CONV_A.TP, FLIP-FLOPA.1Q, SN74LVC1G32A.A
- net DGND: now also C15.2, C18.2, C19.1, C22.1, C8.2, U$11G$1.GND, U$11G$2.NC, U$4G$1.AIN1, U$4G$1.AIN2, U$4G$1.AIN3, U$7.GND; no longer 74LVC1G11G$1.GND, C16.2, C17.1, C21.1, C22.2, C26.2, FLIP-FLOPSUPPLY.GND, GND1.TP, GND2.TP, GND3.TP, SATURATION_DETECTB.GND1, SN74LVC1G32G$1.GND, U$20G$1.!EN, U$20G$1.NO, U$20G$2.GND
- net INPUT_ZERO: now also U$11G$2.IN; no longer U$20G$1.IN
- net N$13: now also R12.1, U$4G$1.AIN0; no longer 74LVC1G11A.Y, SCK.3
- net N$15: now also R4.S; no longer R4.1
- net N$16: now also R11.S, U$11G$2.NO; no longer R10.2, U$20G$1.NC
- net N$19: now also C18.1, DC-DC_CONVERTER.+VOUT, U$8.2; no longer 74LVC1G11A.C, FLIP-FLOPA.1!Q, FLIP-FLOPA.2D
- net N$24: no longer CONV_T.TP
- net N$26: now also SCK.1, SCK_TP.TP; no longer SCK.2, SCK_A.TP
- net SCK_ADC: now also SCK.2; no longer 74LVC1G11A.A, FLIP-FLOPA.1CP, FLIP-FLOPA.2CP, SCK.1, SCK_T.TP
- net SDO_ADC: now also SDA.1, SDA_TP.TP; no longer SDO.1, SDO_A.TP, SN74LVC1G32A.B
- net V_OUT: now also R11.E, R4.A; no longer R10.1, R4.2
Other:
- note added: "+-2.5V"
- note added: "AIN is protected we hav 100 Ohm for limiting"
- note added: "About 4-5 amplification"
- note added: "USE TDN3 1222WISM. Same footprint!!!"
- note removed: "Amplifiaction needs to be defined"
- moved on the sheet: +5V, C2, C22, C25, R3, R5, U$4G$1

Commit message: updated version of board and schematic
Parts:
- added DGND_1, DGND_2: PTR1B1,27, testpad:PTR1B1,27
- added DGND_5, DGND_6: TESTPIN, myLib:TESTPIN
- R12: value 100 -> 1k
- U$11: MOUSER (none) -> 700-MAX4659EUA
Connections:
- net DGND: now also DGND_1.TP, DGND_2.TP, DGND_5.1, DGND_6.1
Other:
- note added: "switched to 757-TCR2EF33LMCT"
- moved on the sheet: C27, CONV_TP, R4, R5, SCK_TP, SDA_TP, U$1G$1, U$3G$1, U$3G$2

Commit message: hw: change isolator to si8400ab
Parts:
- I2C: value ADUM1250 -> SI8400AB-B-IS
Changed lines of the file:
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@@
 <attribute name="DIGIKEY" value="478-7962-1-ND"/>
 </part>
-<part name="I2C" library="ADUM1251WARZ" deviceset="ADUM1251WARZ" device="" value="ADUM1250">
+<part name="I2C" library="ADUM1251WARZ" deviceset="ADUM1251WARZ" device="" value="SI8400AB-B-IS">
 <attribute name="DIGIKEY" value="ADUM1251ARZ-RL7TR-ND"/>
 </part>

Commit message: hw: fix part numbers
Parts:
- I2C: DIGIKEY ADUM1251ARZ-RL7TR-ND -> (none); MOUSER (none) -> 634-SI8400AB-B-IS
Other:
- note added: "Place 2.5V Ref"
Changed lines of the file:
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@@
 </part>
 <part name="I2C" library="ADUM1251WARZ" deviceset="ADUM1251WARZ" device="" value="SI8400AB-B-IS">
-<attribute name="DIGIKEY" value="ADUM1251ARZ-RL7TR-ND"/>
+<attribute name="MOUSER" value="634-SI8400AB-B-IS"/>
 </part>
 <part name="SERIAL_CLOCK" library="ADM2486" deviceset="ADM2486BRWZ-REEL" device="" value="ADM2486BRWZ">
@@
 <text x="320.04" y="208.28" size="1.778" layer="91">+-2.5V</text>
 <text x="365.76" y="299.72" size="1.778" layer="91">switched to 757-TCR2EF33LMCT </text>
+<text x="81.28" y="119.38" size="1.778" layer="91">Place 2.5V Ref</text>
 </plain>
 <instances>
@@
 <attribute name="NAME" x="432.1556" y="100.1014" size="2.0828" layer="95" ratio="6" rot="SMR180"/>
 <attribute name="VALUE" x="431.5206" y="115.3414" size="2.0828" layer="96" ratio="6" rot="SMR180"/>
-<attribute name="DIGIKEY" x="444.5" y="106.68" size="1.778" layer="96" rot="MR180" display="off"/>
+<attribute name="MOUSER" x="444.5" y="106.68" size="1.778" layer="96" rot="MR180" display="off"/>
 </instance>
 <instance part="I2C" gate="G$1" x="419.1" y="370.84" smashed="yes">
