File: hw/kicad/analog-in/analog-in.kicad_sch (KiCad schematic)
At the start: 128 parts

Commit message: update adc to latest version
Parts:
- ADC_0: value LTC2312ITS8-14TRMPBF -> LTC2314-14; DIGIKEY LTC2312CTS8-14#TRMPBFTR-ND -> LTC2314ITS8-14#TRMPBFT-ND
Changed lines of the file:
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@@
       (effects (font (size 1.778 1.5113)) (justify left bottom) hide)
     )
-    (property "Value" "LTC2312ITS8-14TRMPBF" (at 248.6406 326.1614 0)
+    (property "Value" "LTC2314-14" (at 248.6406 326.1614 0)
       (effects (font (size 1.778 1.5113)) (justify left bottom) hide)
     )
@@
       (effects (font (size 1.27 1.27)) hide)
     )
-    (property "DIGIKEY" "LTC2312CTS8-14#TRMPBFTR-ND" (at 261.62 317.5 0)
+    (property "DIGIKEY" "LTC2314ITS8-14#TRMPBFT-ND" (at 261.62 317.5 0)
       (effects (font (size 1.27 1.27)) (justify left bottom) hide)
     )
@@
       (effects (font (size 1.778 1.5113)) (justify left bottom) hide)
     )
-    (property "Value" "LTC2312ITS8-14TRMPBF" (at 246.38 119.38 0)
+    (property "Value" "LTC2314-14" (at 246.38 119.38 0)
       (effects (font (size 1.778 1.5113)) (justify left bottom) hide)
     )
@@
       (effects (font (size 1.27 1.27)) hide)
     )
-    (property "DIGIKEY" "LTC2312CTS8-14#TRMPBFTR-ND" (at 254 106.68 0)
-      (effects (font (size 1.27 1.27)) hide)
-    )
+    (property "DIGIKEY" "LTC2314ITS8-14#TRMPBFT-ND" (at 254 106.68 0)
+      (effects (font (size 1.27 1.27)) hide)
+    )
